File: boards/ShiftOutMosfet/ShiftOutMosfet.kicad_pcb (KiCad board)
At the start: 2 copper layers, 100 x 100 mm, 103 parts, among them J1 CONN_A, J10 CONN_VDD_OUT, J11 CONN_MANUAL, J12 CONN_LOGIC_IN, J13 CONN_LOGIC_OUT, J14 CONN_GNDS, J2 CONN_B, J3 CONN_C, J4 CONN_D, J5 CONN_E, J6 CONN_F, J7 CONN_G, J8 CONN_H, J9 CONN_VDD_IN, Q1 IRL540N, Q2 IRL540N, Q3 IRL540N, Q4 IRL540N, Q5 IRL540N, Q6 IRL540N, Q7 IRL540N, Q8 IRL540N, T1 TEST_LOOP, T10 TEST_LOOP, T11 TEST_LOOP, T12 TEST_LOOP, T13 TEST_LOOP, T14 TEST_LOOP, T15 TEST_LOOP, T16 TEST_LOOP, T2 TEST_LOOP, T3 TEST_LOOP, T4 TEST_LOOP, T5 TEST_LOOP, T6 TEST_LOOP, T7 TEST_LOOP, T8 TEST_LOOP, T9 TEST_LOOP, U1 74HC595

Commit message: Shift mosfet board
Parts:
- removed TP1, TP2, TP3, TP4, TP5, TP6: TEST_LOOP, Virtlink_Misc:TEST_LOOP
- added C1: 100U, Capacitors_THT:CP_Radial_D5.0mm_P2.50mm, F.Cu at (29.8, -12.2)
- added C2: 0.1U, Capacitors_SMD:C_1206_HandSoldering, F.Cu at (25.5, -7.25)
- added C3: C, Capacitors_THT:CP_Radial_D5.0mm_P2.50mm, F.Cu at (54.4, 2.20)
- added D26: 2mA 1.9V, LEDs:LED_1206, F.Cu at (63.2, 9.60)
- added J15: CONN_SIG_OUT, Pin_Headers:Pin_Header_Straight_1x08_Pitch2.54mm, F.Cu at (58.4, -20.3)
- added R34: 10K, Resistors_SMD:R_1206_HandSoldering, F.Cu at (52.4, 18.2)
- added R35: 1K6, Resistors_SMD:R_1206_HandSoldering, F.Cu at (63.4, 17.2)
- added REF**: M3, Virtlink_Hardware:MOUNTINGHOLE_M3, F.Cu at (4.75, -4.75)
- added REF**: M3, Virtlink_Hardware:MOUNTINGHOLE_M3, F.Cu at (95.2, -5.00)
- added T17: TEST_LOOP, Virtlink_Misc:TEST_LOOP, F.Cu at (61.0, 5.20)
- added T18: TEST_LOOP, Virtlink_Misc:TEST_LOOP, F.Cu at (28.4, -19.6)
- added T19: TEST_LOOP, Virtlink_Misc:TEST_LOOP, F.Cu at (56.0, 14.0)
- added T20: TEST_LOOP, Virtlink_Misc:TEST_LOOP, F.Cu at (21.0, -15.6)
- J11: value CONN_MANUAL -> CONN_SIG_IN
- R10, R11, R12, R13, R14, R15, R16, R9: value 250R -> 470K
- U1: footprint Housings_SOIC:SOIC-16_3.9x9.9mm_Pitch1.27mm -> Housings_DIP:DIP-16_W7.62mm_Socket_LongPads
- moved J10 277.1 mm to (-17.6, -66.2)
- moved R23 245.5 mm to (17.2, -36.2)
- moved R31 243.1 mm to (17.2, -30.8)
- moved D7 242.9 mm to (17.2, -59.8), turned to 180 degrees
- moved R15 241.1 mm to (17.2, -41.8), turned to 0 degrees
- moved Q7 240.7 mm to (18.2, -47.2), turned to 90 degrees
- moved T7 240.2 mm to (22.8, -45.8), turned to 90 degrees
- moved T15 239.5 mm to (22.8, -39.2), turned to 90 degrees
- moved J7 239.5 mm to (18.2, -62.8), turned to 270 degrees
- moved D15 238.1 mm to (22.8, -52.2), turned to 90 degrees
- moved D23 237.2 mm to (22.8, -32.8), turned to 90 degrees
- moved R7 235.8 mm to (20.8, -56.8), turned to 180 degrees
- moved R22 227.3 mm to (29.2, -36.2)
- moved D22 225.7 mm to (34.8, -32.8), turned to 90 degrees
- moved R30 223.4 mm to (29.2, -30.8)
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Connections:
- J11 pad 1: /SIG_A -> /A
- J11 pad 2: /SIG_B -> /B
- J11 pad 3: /SIG_C -> /C
- J11 pad 4: /SIG_D -> /D
- J11 pad 5: /SIG_E -> /E
- J11 pad 6: /SIG_F -> /F
- J11 pad 7: /SIG_G -> /G
- J11 pad 8: /SIG_H -> /H
- U1 pad 1: /SIG_B -> /B
- U1 pad 15: /SIG_A -> /A
- U1 pad 2: /SIG_C -> /C
- U1 pad 3: /SIG_D -> /D
- U1 pad 4: /SIG_E -> /E
- U1 pad 5: /SIG_F -> /F
- U1 pad 6: /SIG_G -> /G
- U1 pad 7: /SIG_H -> /H
Routing:
- net VDD: track 18.3 -> 53.0 mm
- net Net-(D16-Pad1): track 0.00 -> 23.2 mm
- net Net-(D15-Pad1): track 0.00 -> 23.2 mm
- net Net-(D14-Pad1): track 0.00 -> 23.2 mm
- net Net-(D13-Pad1): track 0.00 -> 23.2 mm
- net Net-(D12-Pad1): track 0.00 -> 23.2 mm
- net /A: track 0.00 -> 14.8 mm
- net /SIG_A: track 32.6 -> 19.0 mm
- net /SIG_D: track 6.23 -> 18.5 mm
- net /SIG_E: track 6.76 -> 18.5 mm
- net /SIG_F: track 7.89 -> 18.8 mm
- net /SIG_G: track 8.97 -> 18.5 mm
- net /SIG_H: track 10.0 -> 18.5 mm
- net /SIG_B: track 25.1 -> 18.5 mm
- net /D: track 0.00 -> 6.13 mm
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Other:
- board text added: "E"
- board text added: "F"
- board text added: "G"
- board text added: "H"
